Commit message: DF updates
1. Update xacro xml namespace url.
2. Add inertial tags. Values may be incorrect.
3. Add gazebo/material tag combo as traditional URDF material tags don't work.

File: mw_sawppy/urdf/materials.urdf.xacro (robot description, xacro)
@@ -1,4 +1,4 @@
 <?xml version="1.0"?>
-<robot>
+<robot xmlns:xacro="https://www.ros.org/wiki/xacro">
   <!-- Put all the color definitions in a separate file -->
   <material name="Black">

File: mw_sawppy/urdf/sawppy_base.urdf.xacro (robot description, xacro)
@@ -1,4 +1,4 @@
 <?xml version="1.0"?>
-<robot name="base" xmlns:xacro="http://ros.org/wiki/xacro">
+<robot name="base" xmlns:xacro="https://www.ros.org/wiki/xacro">
   <!-- Define a number of dimensions using properties -->
   <xacro:property name="wheel_length" value="0.10" />
@@ -16,4 +16,9 @@
     </joint>
     <link name="${parent}_${suffix}_wheel_link">
+      <inertial>
+        <mass value="0.5"/>
+        <origin xyz="0 0 0" rpy="0 0 0" />
+        <inertia ixx="0.0395416666667" ixy="0" ixz="0" iyy="0.106208333333" iyz="0" izz="0.106208333333"/>
+      </inertial>
       <visual>
         <origin xyz="0 0 0" rpy="0 0 0" />
@@ -24,4 +29,7 @@
       </visual>
     </link>
+    <gazebo reference="${parent}_${suffix}_wheel_link">
+      <material>Gazebo/Black</material>
+    </gazebo>
   </xacro:macro>
   <!-- The base xacro macro -->
@@ -41,4 +49,10 @@
         </geometry>
       </collision>
+      <!-- Inertial properties -->
+      <inertial>
+        <mass value="5"/>
+        <origin rpy="0 0 0" xyz="0 0 0.21"/>
+        <inertia ixx="0.0395416666667" ixy="0" ixz="0" iyy="0.106208333333" iyz="0" izz="0.106208333333"/>
+      </inertial>
     </link>
     <joint name="${name}_joint" type="fixed">
@@ -47,4 +61,7 @@
       <child link="${name}_link" />
     </joint>
+    <gazebo reference="${name}_link">
+      <material>Gazebo/Yellow</material>
+    </gazebo>
   </xacro:macro>
   <link name="base_footprint">

File: mw_sawppy/urdf/sawppy_base_only.xacro (robot description, xacro)
@@ -1,4 +1,4 @@
 <?xml version="1.0"?>
-<robot name="sawppy" xmlns:xacro="http://ros.org/wiki/xacro">
+<robot name="sawppy" xmlns:xacro="https://www.ros.org/wiki/xacro">
    <!-- Include all component files -->
    <xacro:include filename="$(find mw_sawppy)/urdf/materials.urdf.xacro" />
@@ -27,5 +27,13 @@
       </geometry>
     </collision>
+    <inertial>
+      <mass value="0.25"/>
+      <origin rpy="0 0 0" xyz="0 0 0.1"/>
+      <inertia ixx="0.0395416666667" ixy="0" ixz="0" iyy="0.106208333333" iyz="0" izz="0.106208333333"/>
+    </inertial>
   </link>
+  <gazebo reference="t265_model_link">
+    <material>Gazebo/Blue</material>
+  </gazebo>
   <joint name="t265_model_joint" type="fixed">
     <origin xyz="0.215 0 0.275" rpy="0 0 0" />
@@ -47,5 +55,13 @@
       </geometry>
     </collision>
+    <inertial>
+      <mass value="0.25"/>
+      <origin rpy="0 0 0" xyz="0 0 0.1"/>
+      <inertia ixx="0.0395416666667" ixy="0" ixz="0" iyy="0.106208333333" iyz="0" izz="0.106208333333"/>
+    </inertial>
   </link>
+  <gazebo reference="d435_model_link">
+    <material>Gazebo/Blue</material>
+  </gazebo>
   <joint name="d435_model_joint" type="fixed">
     <origin xyz="0.21 0 0.30" rpy="0 0 0" />
