Commit message: Some long forgotten changes

File: mw_sawppy/urdf/sawppy_base_only.xacro (robot description, xacro)
@@ -4,4 +4,5 @@
    <xacro:include filename="$(find mw_sawppy)/urdf/materials.urdf.xacro" />
    <xacro:include filename="$(find mw_sawppy)/urdf/sawppy_base.urdf.xacro" />
+   <xacro:include filename="$(find realsense2_description)/urdf/_d435.urdf.xacro" />
    <!-- Add the base and wheels -->
    <base name="base" color="Yellow"/>
@@ -33,4 +34,8 @@
     <child link="t265_model_link" />
   </joint>
+  <sensor_d435 parent="base_link">
+    <origin xyz="0.21 0 0.30" rpy="0 0 0"/>
+  </sensor_d435>
+  <!--
   <link name="d435_model_link">
     <visual>
@@ -53,4 +58,5 @@
     <child link="d435_model_link" />
   </joint>
+  -->
   <virtual_joint name="base_odom" type="planar" parent_frame="odom" child_link="base_footprint" />
 </robot>
